File: IO.sch (KiCad schematic (older format))
At the start: 40 parts, among them J10 Conn_01x03, J12 Conn_01x03, J13 Conn_01x03, J14 Conn_01x03, J15 Conn_01x03, J17 Conn_01x03, J18 Conn_01x03, J19 Conn_01x03, J2 Conn_01x03, J20 Conn_01x03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

Commit message: Update
Parts:
- C10: LCSC Part # (none) -> C15525
- R11, R12: LCSC Part # (none) -> C25744
- R15, R16, R17, R18, R19, R20, R21, R22, R23, R24, R25, R26, R27, R28, R29, R30: LCSC Part # (none) -> C1555
- U2: LCSC Part # (none) -> C92206
Changed lines of the file:
@@
 F 2 "Package_SO:TSSOP-28_4.4x9.7mm_P0.65mm" H 2625 5525 50  0001 L CNN
 F 3 "http://www.nxp.com/documents/data_sheet/PCA9685.pdf" H 2200 7200 50  0001 C CNN
+F 4 "C92206" H 2600 6500 50  0001 C CNN "LCSC Part #"
 	1    2600 6500
 	1    0    0    -1
@@
 F 2 "Resistor_SMD:R_0402_1005Metric" H 1750 6250 50  0001 C CNN
 F 3 "~" H 1750 6250 50  0001 C CNN
+F 4 "C25744" H 1750 6250 50  0001 C CNN "LCSC Part #"
 	1    1750 6250
 	1    0    0    -1
@@
 F 2 "Capacitor_SMD:C_0402_1005Metric" H 2900 5350 50  0001 C CNN
 F 3 "~" H 2900 5350 50  0001 C CNN
+F 4 "C15525" H 2900 5350 50  0001 C CNN "LCSC Part #"
 	1    2900 5350
 	1    0    0    -1
@@
 F 2 "Resistor_SMD:R_0402_1005Metric" H 1600 7200 50  0001 C CNN
 F 3 "~" H 1600 7200 50  0001 C CNN
+F 4 "C25744" H 1600 7200 50  0001 C CNN "LCSC Part #"
 	1    1600 7200
 	0    1    1    0
@@
 F 2 "Resistor_SMD:R_0402_1005Metric" H 4500 5850 50  0001 C CNN
 F 3 "~" H 4500 5850 50  0001 C CNN
+F 4 "C1555" H 4500 5850 50  0001 C CNN "LCSC Part #"
 	1    4500 5850
 	0    -1   1    0
@@
 F 2 "Resistor_SMD:R_0402_1005Metric" H 4500 5700 50  0001 C CNN
 F 3 "~" H 4500 5700 50  0001 C CNN
+F 4 "C1555" H 4500 5700 50  0001 C CNN "LCSC Part #"
 	1    4500 5700
 	0    -1   1    0
@@
 F 2 "Resistor_SMD:R_0402_1005Metric" H 4500 5550 50  0001 C CNN
 F 3 "~" H 4500 5550 50  0001 C CNN
+F 4 "C1555" H 4500 5550 50  0001 C CNN "LCSC Part #"
 	1    4500 5550
 	0    -1   1    0
@@
 F 2 "Resistor_SMD:R_0402_1005Metric" H 4500 5400 50  0001 C CNN
 F 3 "~" H 4500 5400 50  0001 C CNN
+F 4 "C1555" H 4500 5400 50  0001 C CNN "LCSC Part #"
 	1    4500 5400
 	0    -1   1    0
@@
 F 2 "Resistor_SMD:R_0402_1005Metric" H 4500 6000 50  0001 C CNN
 F 3 "~" H 4500 6000 50  0001 C CNN
+F 4 "C1555" H 4500 6000 50  0001 C CNN "LCSC Part #"
 	1    4500 6000
 	0    -1   -1   0
@@
 F 2 "Resistor_SMD:R_0402_1005Metric" H 4500 6150 50  0001 C CNN
 F 3 "~" H 4500 6150 50  0001 C CNN
+F 4 "C1555" H 4500 6150 50  0001 C CNN "LCSC Part #"
 	1    4500 6150
 	0    -1   -1   0
@@
 F 2 "Resistor_SMD:R_0402_1005Metric" H 4500 6300 50  0001 C CNN
 F 3 "~" H 4500 6300 50  0001 C CNN
+F 4 "C1555" H 4500 6300 50  0001 C CNN "LCSC Part #"
 	1    4500 6300
 	0    -1   -1   0
@@
 F 2 "Resistor_SMD:R_0402_1005Metric" H 4500 6450 50  0001 C CNN
 F 3 "~" H 4500 6450 50  0001 C CNN
+F 4 "C1555" H 4500 6450 50  0001 C CNN "LCSC Part #"
 	1    4500 6450
 	0    -1   -1   0
@@
 F 2 "Resistor_SMD:R_0402_1005Metric" H 4500 7650 50  0001 C CNN
 F 3 "~" H 4500 7650 50  0001 C CNN
+F 4 "C1555" H 4500 7650 50  0001 C CNN "LCSC Part #"
 	1    4500 7650
 	0    -1   1    0
@@
 F 2 "Resistor_SMD:R_0402_1005Metric" H 4500 7500 50  0001 C CNN
 F 3 "~" H 4500 7500 50  0001 C CNN
+F 4 "C1555" H 4500 7500 50  0001 C CNN "LCSC Part #"
 	1    4500 7500
 	0    -1   1    0
@@
 F 2 "Resistor_SMD:R_0402_1005Metric" H 4500 7350 50  0001 C CNN
 F 3 "~" H 4500 7350 50  0001 C CNN
+F 4 "C1555" H 4500 7350 50  0001 C CNN "LCSC Part #"
 	1    4500 7350
 	0    -1   1    0
@@
 F 2 "Resistor_SMD:R_0402_1005Metric" H 4500 7200 50  0001 C CNN
 F 3 "~" H 4500 7200 50  0001 C CNN
+F 4 "C1555" H 4500 7200 50  0001 C CNN "LCSC Part #"
 	1    4500 7200
 	0    -1   1    0
@@
 F 2 "Resistor_SMD:R_0402_1005Metric" H 4500 6600 50  0001 C CNN
 F 3 "~" H 4500 6600 50  0001 C CNN
+F 4 "C1555" H 4500 6600 50  0001 C CNN "LCSC Part #"
 	1    4500 6600
 	0    -1   -1   0
@@
 F 2 "Resistor_SMD:R_0402_1005Metric" H 4500 6750 50  0001 C CNN
 F 3 "~" H 4500 6750 50  0001 C CNN
+F 4 "C1555" H 4500 6750 50  0001 C CNN "LCSC Part #"
 	1    4500 6750
 	0    -1   -1   0
@@
 F 2 "Resistor_SMD:R_0402_1005Metric" H 4500 6900 50  0001 C CNN
 F 3 "~" H 4500 6900 50  0001 C CNN
+F 4 "C1555" H 4500 6900 50  0001 C CNN "LCSC Part #"
 	1    4500 6900
 	0    -1   -1   0
@@
 F 2 "Resistor_SMD:R_0402_1005Metric" H 4500 7050 50  0001 C CNN
 F 3 "~" H 4500 7050 50  0001 C CNN
+F 4 "C1555" H 4500 7050 50  0001 C CNN "LCSC Part #"
 	1    4500 7050
 	0    -1   -1   0
