File: Main.sch (KiCad schematic (older format))
At the start: 31 parts, among them J25 SWD, J26 5v In, J27 LCD, J28 USART2, J29 USART3, J30 3557-2, SW2 Reset, U1 STM32F103RBT6, U3 AZ1117-3.3, Y1 Crystal_GND24

Commit message: Update
Parts:
- C1, C3: LCSC Part # (none) -> C1547
- C11: LCSC Part # (none) -> C52923
- C12, C13, C2, C5, C6, C7, C8, C9: LCSC Part # (none) -> C1525
- C4: LCSC Part # (none) -> C23733
- D9: LCSC Part # (none) -> C2286
- R1, R2: LCSC Part # (none) -> C25900
- R3: LCSC Part # (none) -> C25879
- R4: LCSC Part # (none) -> C25118
- U1: LCSC Part # (none) -> C8735
- U3: LCSC Part # (none) -> C6186
- Y1: LCSC Part # (none) -> C13738
Changed lines of the file:
@@
 $Descr USLetter 11000 8500
 encoding utf-8
-Sheet 2 4
+Sheet 4 4
 Title "ALP Control Board"
 Date "2020-10-09"
@@
 F 2 "Capacitor_SMD:C_0402_1005Metric" H 4200 1050 50  0001 C CNN
 F 3 "~" H 4200 1050 50  0001 C CNN
+F 4 "C23733" H 4200 1050 50  0001 C CNN "LCSC Part #"
 	1    4200 1050
 	1    0    0    -1
@@
 F 2 "Capacitor_SMD:C_0402_1005Metric" H 4700 1050 50  0001 C CNN
 F 3 "~" H 4700 1050 50  0001 C CNN
+F 4 "C1525" H 4700 1050 50  0001 C CNN "LCSC Part #"
 	1    4700 1050
 	1    0    0    -1
@@
 F 2 "Capacitor_SMD:C_0402_1005Metric" H 5200 1050 50  0001 C CNN
 F 3 "~" H 5200 1050 50  0001 C CNN
+F 4 "C1525" H 5200 1050 50  0001 C CNN "LCSC Part #"
 	1    5200 1050
 	1    0    0    -1
@@
 F 2 "Capacitor_SMD:C_0402_1005Metric" H 5700 1050 50  0001 C CNN
 F 3 "~" H 5700 1050 50  0001 C CNN
+F 4 "C1525" H 5700 1050 50  0001 C CNN "LCSC Part #"
 	1    5700 1050
 	1    0    0    -1
@@
 F 2 "Capacitor_SMD:C_0402_1005Metric" H 6200 1050 50  0001 C CNN
 F 3 "~" H 6200 1050 50  0001 C CNN
+F 4 "C1525" H 6200 1050 50  0001 C CNN "LCSC Part #"
 	1    6200 1050
 	1    0    0    -1
@@
 F 2 "Capacitor_SMD:C_0402_1005Metric" H 1800 3400 50  0001 C CNN
 F 3 "~" H 1800 3400 50  0001 C CNN
+F 4 "C1547" H 1800 3400 50  0001 C CNN "LCSC Part #"
 	1    1800 3400
 	1    0    0    -1
@@
 F 2 "Resistor_SMD:R_0402_1005Metric" H 1800 3000 50  0001 C CNN
 F 3 "~" H 1800 3000 50  0001 C CNN
+F 4 "C25118" H 1800 3000 50  0001 C CNN "LCSC Part #"
 	1    1800 3000
 	-1   0    0    1
@@
 F 2 "Crystal:Crystal_SMD_3225-4Pin_3.2x2.5mm" H 1550 3200 50  0001 C CNN
 F 3 "~" H 1550 3200 50  0001 C CNN
+F 4 "C13738" H 1550 3200 50  0001 C CNN "LCSC Part #"
 	1    1550 3200
 	1    0    0    -1
@@
 F 2 "Capacitor_SMD:C_0402_1005Metric" H 1300 3400 50  0001 C CNN
 F 3 "~" H 1300 3400 50  0001 C CNN
+F 4 "C1547" H 1300 3400 50  0001 C CNN "LCSC Part #"
 	1    1300 3400
 	1    0    0    -1
@@
 F 2 "Capacitor_SMD:C_0402_1005Metric" H 1700 1400 50  0001 C CNN
 F 3 "~" H 1700 1400 50  0001 C CNN
+F 4 "C1525" H 1700 1400 50  0001 C CNN "LCSC Part #"
 	1    1700 1400
 	1    0    0    -1
@@
 F 2 "Capacitor_SMD:C_0402_1005Metric" H 6700 1050 50  0001 C CNN
 F 3 "~" H 6700 1050 50  0001 C CNN
+F 4 "C1525" H 6700 1050 50  0001 C CNN "LCSC Part #"
 	1    6700 1050
 	1    0    0    -1
@@
 F 2 "Package_QFP:LQFP-64_10x10mm_P0.5mm" H 6350 2650 50  0001 R CNN
 F 3 "http://www.st.com/st-web-ui/static/active/en/resource/technical/document/datasheet/CD00161566.pdf" H 6950 4350 50  0001 C CNN
+F 4 "C8735" H 6950 4350 50  0001 C CNN "LCSC Part #"
 	1    6950 4350
 	1    0    0    -1
@@
 F 2 "Capacitor_SMD:C_0402_1005Metric" H 7200 1050 50  0001 C CNN
 F 3 "~" H 7200 1050 50  0001 C CNN
+F 4 "C52923" H 7200 1050 50  0001 C CNN "LCSC Part #"
 	1    7200 1050
 	-1   0    0    1
@@
 F 2 "Resistor_SMD:R_0402_1005Metric" H 1400 5550 50  0001 C CNN
 F 3 "~" H 1400 5550 50  0001 C CNN
+F 4 "C25900" H 1400 5550 50  0001 C CNN "LCSC Part #"
 	1    1400 5550
 	0    -1   -1   0
@@
 F 2 "Resistor_SMD:R_0402_1005Metric" H 1400 5200 50  0001 C CNN
 F 3 "~" H 1400 5200 50  0001 C CNN
+F 4 "C25900" H 1400 5200 50  0001 C CNN "LCSC Part #"
 	1    1400 5200
 	0    -1   -1   0
@@
 F 2 "Package_TO_SOT_SMD:SOT-223-3_TabPin2" H 4000 4700 50  0001 C CIN
 F 3 "https://www.diodes.com/assets/Datasheets/AZ1117.pdf" H 4000 4450 50  0001 C CNN
+F 4 "C6186" H 4000 4450 50  0001 C CNN "LCSC Part #"
 	1    4000 4450
 	1    0    0    -1
@@
 F 2 "Capacitor_SMD:C_0402_1005Metric" H 3400 4850 50  0001 C CNN
 F 3 "~" H 3400 4850 50  0001 C CNN
+F 4 "C1525" H 3400 4850 50  0001 C CNN "LCSC Part #"
 	1    3400 4850
 	1    0    0    -1
@@
 F 2 "Capacitor_SMD:C_0402_1005Metric" H 4550 4850 50  0001 C CNN
 F 3 "~" H 4550 4850 50  0001 C CNN
+F 4 "C1525" H 4550 4850 50  0001 C CNN "LCSC Part #"
 	1    4550 4850
 	1    0    0    -1
@@
 F 2 "LED_SMD:LED_0603_1608Metric" H 3900 6800 50  0001 C CNN
 F 3 "~" H 3900 6800 50  0001 C CNN
+F 4 "C2286" H 3900 6800 50  0001 C CNN "LCSC Part #"
 	1    3900 6800
 	0    -1   -1   0
@@
 F 2 "Resistor_SMD:R_0402_1005Metric" H 3900 7150 50  0001 C CNN
 F 3 "~" H 3900 7150 50  0001 C CNN
+F 4 "C25879" H 3900 7150 50  0001 C CNN "LCSC Part #"
 	1    3900 7150
 	1    0    0    -1
