File: Relays.sch (KiCad schematic (older format))
At the start: 40 parts, among them J1 Out0, J11 Out1, J16 Out5, J21 Out2, J22 Out6, J23 Out3, J24 Out7, J6 Out4, Q1 BFS20, Q2 BFS20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

Commit message: Update
Parts:
- D1, D2, D3, D4, D5, D6, D7, D8: value 1N4001 -> B5819W; LCSC Part # (none) -> C8598
- Q1, Q2, Q3, Q4, Q5, Q6, Q7, Q8: value BFS20 -> MMBT3904; LCSC Part # (none) -> C20526
- R10, R13, R14, R5, R6, R7, R8, R9: LCSC Part # (none) -> C11702
Changed lines of the file:
@@
 $Descr A4 11693 8268
 encoding utf-8
-Sheet 4 4
+Sheet 3 4
 Title "ALP Control Board"
 Date "2020-10-09"
@@
 AR Path="/5FE183FC/5FE1890B" Ref="Q1"  Part="1"
 F 0 "Q1" H 1800 2450 50  0000 L CNN
-F 1 "BFS20" H 1650 2550 50  0000 L CNN
+F 1 "MMBT3904" H 1650 2550 50  0000 L CNN
 F 2 "Package_TO_SOT_SMD:SOT-23" H 2050 2850 50  0001 C CNN
 F 3 "~" H 1850 2750 50  0001 C CNN
+F 4 "C20526" H 1850 2750 50  0001 C CNN "LCSC Part #"
 	1    1850 2750
 	-1   0    0    -1
@@
 F 2 "Resistor_SMD:R_0402_1005Metric" H 2150 2750 50  0001 C CNN
 F 3 "~" H 2150 2750 50  0001 C CNN
+F 4 "C11702" H 2150 2750 50  0001 C CNN "LCSC Part #"
 	1    2150 2750
 	0    -1   1    0
@@
 AR Path="/5FE183FC/5FE18A95" Ref="D1"  Part="1"
 F 0 "D1" V 1650 2050 50  0000 L CNN
-F 1 "1N4001" V 1750 1950 50  0000 L CNN
+F 1 "B5819W" V 1750 1950 50  0000 L CNN
 F 2 "Diode_SMD:D_SOD-123" H 1650 2075 50  0001 C CNN
 F 3 "http://www.vishay.com/docs/88503/1n4001.pdf" H 1650 2250 50  0001 C CNN
 F 4 "C81598" V 1650 2250 50  0001 C CNN "LCSC PN"
+F 5 "C8598" H 1650 2250 50  0001 C CNN "LCSC Part #"
 	1    1650 2250
 	0    1    1    0
@@
 AR Path="/5FE183FC/5FE5F4CC" Ref="Q3"  Part="1"
 F 0 "Q3" H 3950 2450 50  0000 L CNN
-F 1 "BFS20" H 3800 2550 50  0000 L CNN
+F 1 "MMBT3904" H 3800 2550 50  0000 L CNN
 F 2 "Package_TO_SOT_SMD:SOT-23" H 4200 2850 50  0001 C CNN
 F 3 "~" H 4000 2750 50  0001 C CNN
+F 4 "C20526" H 4000 2750 50  0001 C CNN "LCSC Part #"
 	1    4000 2750
 	-1   0    0    -1
@@
 F 2 "Resistor_SMD:R_0402_1005Metric" H 4300 2750 50  0001 C CNN
 F 3 "~" H 4300 2750 50  0001 C CNN
+F 4 "C11702" H 4300 2750 50  0001 C CNN "LCSC Part #"
 	1    4300 2750
 	0    -1   1    0
@@
 AR Path="/5FE183FC/5FE5F4EC" Ref="D3"  Part="1"
 F 0 "D3" V 3800 2050 50  0000 L CNN
-F 1 "1N4001" V 3900 1950 50  0000 L CNN
+F 1 "B5819W" V 3900 1950 50  0000 L CNN
 F 2 "Diode_SMD:D_SOD-123" H 3800 2075 50  0001 C CNN
 F 3 "http://www.vishay.com/docs/88503/1n4001.pdf" H 3800 2250 50  0001 C CNN
 F 4 "C81598" V 3800 2250 50  0001 C CNN "LCSC PN"
+F 5 "C8598" H 3800 2250 50  0001 C CNN "LCSC Part #"
 	1    3800 2250
 	0    1    1    0
@@
 AR Path="/5FE183FC/5FE5F941" Ref="Q5"  Part="1"
 F 0 "Q5" H 6200 2450 50  0000 L CNN
-F 1 "BFS20" H 6050 2550 50  0000 L CNN
+F 1 "MMBT3904" H 6050 2550 50  0000 L CNN
 F 2 "Package_TO_SOT_SMD:SOT-23" H 6450 2850 50  0001 C CNN
 F 3 "~" H 6250 2750 50  0001 C CNN
+F 4 "C20526" H 6250 2750 50  0001 C CNN "LCSC Part #"
 	1    6250 2750
 	-1   0    0    -1
@@
 F 2 "Resistor_SMD:R_0402_1005Metric" H 6550 2750 50  0001 C CNN
 F 3 "~" H 6550 2750 50  0001 C CNN
+F 4 "C11702" H 6550 2750 50  0001 C CNN "LCSC Part #"
 	1    6550 2750
 	0    -1   1    0
@@
 AR Path="/5FE183FC/5FE5F964" Ref="D5"  Part="1"
 F 0 "D5" V 6050 2050 50  0000 L CNN
-F 1 "1N4001" V 6150 1950 50  0000 L CNN
+F 1 "B5819W" V 6150 1950 50  0000 L CNN
 F 2 "Diode_SMD:D_SOD-123" H 6050 2075 50  0001 C CNN
 F 3 "http://www.vishay.com/docs/88503/1n4001.pdf" H 6050 2250 50  0001 C CNN
 F 4 "C81598" V 6050 2250 50  0001 C CNN "LCSC PN"
+F 5 "C8598" H 6050 2250 50  0001 C CNN "LCSC Part #"
 	1    6050 2250
 	0    1    1    0
@@
 AR Path="/5FE183FC/5FE6060C" Ref="Q7"  Part="1"
 F 0 "Q7" H 8600 2450 50  0000 L CNN
-F 1 "BFS20" H 8450 2550 50  0000 L CNN
+F 1 "MMBT3904" H 8450 2550 50  0000 L CNN
 F 2 "Package_TO_SOT_SMD:SOT-23" H 8850 2850 50  0001 C CNN
 F 3 "~" H 8650 2750 50  0001 C CNN
+F 4 "C20526" H 8650 2750 50  0001 C CNN "LCSC Part #"
 	1    8650 2750
 	-1   0    0    -1
@@
 F 2 "Resistor_SMD:R_0402_1005Metric" H 8950 2750 50  0001 C CNN
 F 3 "~" H 8950 2750 50  0001 C CNN
+F 4 "C11702" H 8950 2750 50  0001 C CNN "LCSC Part #"
 	1    8950 2750
 	0    -1   1    0
@@
 AR Path="/5FE183FC/5FE6062F" Ref="D7"  Part="1"
 F 0 "D7" V 8450 2050 50  0000 L CNN
-F 1 "1N4001" V 8550 1950 50  0000 L CNN
+F 1 "B5819W" V 8550 1950 50  0000 L CNN
 F 2 "Diode_SMD:D_SOD-123" H 8450 2075 50  0001 C CNN
 F 3 "http://www.vishay.com/docs/88503/1n4001.pdf" H 8450 2250 50  0001 C CNN
 F 4 "C81598" V 8450 2250 50  0001 C CNN "LCSC PN"
+F 5 "C8598" H 8450 2250 50  0001 C CNN "LCSC Part #"
 	1    8450 2250
 	0    1    1    0
@@
 AR Path="/5FE183FC/5FE612A0" Ref="Q2"  Part="1"
 F 0 "Q2" H 1800 4650 50  0000 L CNN
-F 1 "BFS20" H 1650 4750 50  0000 L CNN
+F 1 "MMBT3904" H 1650 4750 50  0000 L CNN
 F 2 "Package_TO_SOT_SMD:SOT-23" H 2050 5050 50  0001 C CNN
 F 3 "~" H 1850 4950 50  0001 C CNN
+F 4 "C20526" H 1850 4950 50  0001 C CNN "LCSC Part #"
 	1    1850 4950
 	-1   0    0    -1
@@
 F 2 "Resistor_SMD:R_0402_1005Metric" H 2150 4950 50  0001 C CNN
 F 3 "~" H 2150 4950 50  0001 C CNN
+F 4 "C11702" H 2150 4950 50  0001 C CNN "LCSC Part #"
 	1    2150 4950
 	0    -1   1    0
@@
 AR Path="/5FE183FC/5FE612C0" Ref="D2"  Part="1"
 F 0 "D2" V 1650 4250 50  0000 L CNN
-F 1 "1N4001" V 1750 4150 50  0000 L CNN
+F 1 "B5819W" V 1750 4150 50  0000 L CNN
 F 2 "Diode_SMD:D_SOD-123" H 1650 4275 50  0001 C CNN
 F 3 "http://www.vishay.com/docs/88503/1n4001.pdf" H 1650 4450 50  0001 C CNN
 F 4 "C81598" V 1650 4450 50  0001 C CNN "LCSC PN"
+F 5 "C8598" H 1650 4450 50  0001 C CNN "LCSC Part #"
 	1    1650 4450
 	0    1    1    0
@@
 AR Path="/5FE183FC/5FE612DC" Ref="Q4"  Part="1"
 F 0 "Q4" H 3950 4650 50  0000 L CNN
-F 1 "BFS20" H 3800 4750 50  0000 L CNN
+F 1 "MMBT3904" H 3800 4750 50  0000 L CNN
 F 2 "Package_TO_SOT_SMD:SOT-23" H 4200 5050 50  0001 C CNN
 F 3 "~" H 4000 4950 50  0001 C CNN
+F 4 "C20526" H 4000 4950 50  0001 C CNN "LCSC Part #"
 	1    4000 4950
 	-1   0    0    -1
@@
 F 2 "Resistor_SMD:R_0402_1005Metric" H 4300 4950 50  0001 C CNN
 F 3 "~" H 4300 4950 50  0001 C CNN
+F 4 "C11702" H 4300 4950 50  0001 C CNN "LCSC Part #"
 	1    4300 4950
 	0    -1   1    0
@@
 AR Path="/5FE183FC/5FE612FC" Ref="D4"  Part="1"
 F 0 "D4" V 3800 4250 50  0000 L CNN
-F 1 "1N4001" V 3900 4150 50  0000 L CNN
+F 1 "B5819W" V 3900 4150 50  0000 L CNN
 F 2 "Diode_SMD:D_SOD-123" H 3800 4275 50  0001 C CNN
 F 3 "http://www.vishay.com/docs/88503/1n4001.pdf" H 3800 4450 50  0001 C CNN
 F 4 "C81598" V 3800 4450 50  0001 C CNN "LCSC PN"
+F 5 "C8598" H 3800 4450 50  0001 C CNN "LCSC Part #"
 	1    3800 4450
 	0    1    1    0
@@
 AR Path="/5FE183FC/5FE61318" Ref="Q6"  Part="1"
 F 0 "Q6" H 6200 4650 50  0000 L CNN
-F 1 "BFS20" H 6050 4750 50  0000 L CNN
+F 1 "MMBT3904" H 6050 4750 50  0000 L CNN
 F 2 "Package_TO_SOT_SMD:SOT-23" H 6450 5050 50  0001 C CNN
 F 3 "~" H 6250 4950 50  0001 C CNN
+F 4 "C20526" H 6250 4950 50  0001 C CNN "LCSC Part #"
 	1    6250 4950
 	-1   0    0    -1
@@
 F 2 "Resistor_SMD:R_0402_1005Metric" H 6550 4950 50  0001 C CNN
 F 3 "~" H 6550 4950 50  0001 C CNN
+F 4 "C11702" H 6550 4950 50  0001 C CNN "LCSC Part #"
 	1    6550 4950
 	0    -1   1    0
@@
 AR Path="/5FE183FC/5FE61338" Ref="D6"  Part="1"
 F 0 "D6" V 6050 4250 50  0000 L CNN
-F 1 "1N4001" V 6150 4150 50  0000 L CNN
+F 1 "B5819W" V 6150 4150 50  0000 L CNN
 F 2 "Diode_SMD:D_SOD-123" H 6050 4275 50  0001 C CNN
 F 3 "http://www.vishay.com/docs/88503/1n4001.pdf" H 6050 4450 50  0001 C CNN
 F 4 "C81598" V 6050 4450 50  0001 C CNN "LCSC PN"
+F 5 "C8598" H 6050 4450 50  0001 C CNN "LCSC Part #"
 	1    6050 4450
 	0    1    1    0
@@
 AR Path="/5FE183FC/5FE61355" Ref="Q8"  Part="1"
 F 0 "Q8" H 8600 4650 50  0000 L CNN
-F 1 "BFS20" H 8450 4750 50  0000 L CNN
+F 1 "MMBT3904" H 8450 4750 50  0000 L CNN
 F 2 "Package_TO_SOT_SMD:SOT-23" H 8850 5050 50  0001 C CNN
 F 3 "~" H 8650 4950 50  0001 C CNN
+F 4 "C20526" H 8650 4950 50  0001 C CNN "LCSC Part #"
 	1    8650 4950
 	-1   0    0    -1
@@
 F 2 "Resistor_SMD:R_0402_1005Metric" H 8950 4950 50  0001 C CNN
 F 3 "~" H 8950 4950 50  0001 C CNN
+F 4 "C11702" H 8950 4950 50  0001 C CNN "LCSC Part #"
 	1    8950 4950
 	0    -1   1    0
@@
 AR Path="/5FE183FC/5FE61375" Ref="D8"  Part="1"
 F 0 "D8" V 8450 4250 50  0000 L CNN
-F 1 "1N4001" V 8550 4150 50  0000 L CNN
+F 1 "B5819W" V 8550 4150 50  0000 L CNN
 F 2 "Diode_SMD:D_SOD-123" H 8450 4275 50  0001 C CNN
 F 3 "http://www.vishay.com/docs/88503/1n4001.pdf" H 8450 4450 50  0001 C CNN
 F 4 "C81598" V 8450 4450 50  0001 C CNN "LCSC PN"
+F 5 "C8598" H 8450 4450 50  0001 C CNN "LCSC Part #"
 	1    8450 4450
 	0    1    1    0
